File: Board design/Cowbell.kicad_pcb (KiCad board)
At the start: 2 copper layers, 23.7 x 53.5 mm, 25 parts, among them J1 Conn_Coaxial, J101 Conn_Coaxial, J102 Conn_01x02_Male, J104 Conn_01x02_Male, J105 Conn_01x02_Male, U101 NEO-M8, U102 LSM303C, U103 ESP32-WROOM-32, U104 RN2483A-I

Commit message: Add files via upload
Routing:
- net SCL: track 46.6 -> 43.4 mm
- net Tx0: track 17.9 -> 20.3 mm
- net /VccGPS_backup: track 18.7 -> 21.0 mm
- net Net-(J105-Pad1): track 28.5 -> 30.7 mm
- net SDA: track 47.4 -> 45.8 mm
- net Rx0: track 14.0 -> 15.6 mm
- net Tx1: track 9.92 -> 8.39 mm
- net Rx1: track 8.66 -> 7.74 mm
- net Net-(C202-Pad1): track 25.2 -> 24.4 mm
- net /VCC103: track 40.0 -> 39.3 mm
- net Timepulse: track 29.1 -> 28.4 mm
- net GND: vias 80 -> 82
Other:
- rule via_min_drill: 0.254 -> 0.305
- board text added: "+ Batt -"
- board text added: "BackUp Batt"
- board text removed: "18650?"

Commit message: Add files via upload
skifte til sim28
Parts:
- removed J101: Conn_Coaxial, Connectors_Molex:Molex_SMA_Jack_Edge_Mount
- removed R1: DNC, Resistors_SMD:R_0603_HandSoldering
- removed R103, R104, R105, R107: 2k2, Resistors_SMD:R_0603
- removed R106: 10k, Resistors_SMD:R_0603
- added J401: Conn_Coaxial, Emborg:SMA_EdgeMount, B.Cu at (125.9, 27.9)
- added L101: >27nH, Inductor_SMD:L_0402_1005Metric, F.Cu at (119.8, 69.7)
- added Q102: DMG6601LVT, Emborg:DMG6601LVT, B.Cu at (122.8, 70.2)
- added R302: 2k2, Resistor_SMD:R_0603_1608Metric, F.Cu at (132.0, 67.6)
- added R307: 2k2, Resistor_SMD:R_0603_1608Metric, B.Cu at (118.5, 35.5)
- added R401: 10k, Resistor_SMD:R_0603_1608Metric, B.Cu at (137.9, 45.2)
- R101: footprint Resistors_SMD:R_0603_HandSoldering -> Resistor_SMD:R_0603_1608Metric_Pad1.05x0.95mm_HandSolder
- R102: value 2k2 -> 10ohm; footprint Resistors_SMD:R_0603 -> Resistor_SMD:R_0603_1608Metric_Pad1.05x0.95mm_HandSolder; moved to F.Cu
- R201, R202: footprint Resistors_SMD:R_0603 -> Resistor_SMD:R_0603_1608Metric
- U101: value NEO-M8 -> SIM28ML; footprint Emborg:NEO-M8 -> Emborg:SIM28ML
- moved R101 26.1 mm to (123.3, 66.6), turned to 0 degrees
- moved R202 20.3 mm to (130.8, 57.5), turned to 180 degrees
- moved R201 20.0 mm to (133.9, 57.5), turned to 180 degrees
- moved C201 17.5 mm to (129.8, 60.2), turned to 270 degrees
- moved H101 16.8 mm to (118.6, 28.8)
- moved U102 16.4 mm to (132.3, 60.2), turned to 270 degrees
- moved J1 13.8 mm to (119.3, 73.7)
- moved BT101 13.6 mm to (130.9, 73.2)
- moved C203 12.9 mm to (132.3, 62.7), turned to 180 degrees
- moved C204 11.5 mm to (134.9, 63.5), turned to 270 degrees
- moved C202 11.1 mm to (132.1, 64.1), turned to 180 degrees
- moved J102 10.4 mm to (127.4, 72.0), turned to 0 degrees
- moved U101 4.75 mm to (122.6, 61.5)
- moved R102 4.10 mm to (122.8, 69.9), turned to 0 degrees
- moved J104 0.76 mm to (136.2, 31.4)
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Connections:
- C202 pad 1: Net-(C202-Pad1) -> +3V3
- C203 pad 1: Net-(C202-Pad1) -> +3V3
- C204 pad 1: Net-(C202-Pad1) -> +3V3
- R101 pad 1: /VCC102 -> Net-(Q102-Pad2)
- R101 pad 2: Net-(R101-Pad2) -> Net-(Q102-Pad3)
- R102 pad 1: /VCC103 -> Net-(L101-Pad2)
- R102 pad 2: Net-(J105-Pad1) -> Net-(Q102-Pad4)
- R201 pad 2: Net-(C202-Pad1) -> +3V3
- R202 pad 1: Net-(C202-Pad1) -> +3V3
- U101 pad 1: Net-(U101-Pad1) -> GND
- U101 pad 13: GND -> Net-(Q102-Pad1)
- U101 pad 14: Net-(U101-Pad14) -> Net-(Q102-Pad2)
- U101 pad 2: Net-(U101-Pad2) -> Tx0
- U101 pad 3: Timepulse -> Rx0
- U101 pad 4: Extint -> Timepulse
- U101 pad 6: Net-(U101-Pad6) -> /VccGPS_backup
- U101 pad 8: Net-(R1-Pad2) -> +3V3
- U102 pad 10: Net-(C202-Pad1) -> +3V3
- U102 pad 2: Net-(C202-Pad1) -> +3V3
- U102 pad 3: Net-(C202-Pad1) -> +3V3
- U102 pad 9: Net-(C202-Pad1) -> +3V3
- U103 pad 2: /VCC103 -> +3V3
- U104 pad 12: /VCC102 -> +3V3
- U104 pad 32: Net-(R101-Pad2) -> Net-(R401-Pad2)
- U104 pad 34: /VCC102 -> +3V3
Routing:
- net +3V3: track 10.4 -> 144.2 mm, vias 0 -> 6
- net /VCC102: track 40.9 -> 0.00 mm
- net /VCC103: track 39.3 -> 0.00 mm, vias 2 -> 0
- net GND: track 107.4 -> 72.9 mm, vias 82 -> 81
- net Extint: track 26.9 -> 0.00 mm, vias 2 -> 0
- net Net-(C202-Pad1): track 24.4 -> 0.00 mm, vias 1 -> 0
- net SDA: track 45.8 -> 26.5 mm
- net Int_MAG: track 35.4 -> 20.1 mm
- net SCL: track 43.4 -> 30.1 mm
- net /VCC101: track 12.0 -> 0.00 mm, vias 2 -> 0
- net Timepulse: track 28.4 -> 18.4 mm
- net Net-(J105-Pad1): track 30.7 -> 23.3 mm, vias 3 -> 0
- net Int_XL: track 33.1 -> 26.3 mm
- net Net-(Q102-Pad3): track 0.00 -> 6.46 mm
- net Net-(R1-Pad2): track 4.87 -> 0.00 mm
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Other:
- board size 23.7 x 53.5 mm -> 23.7 x 52.5 mm
- board text added: "GPS SIM28ml"
- board text removed: "GPS NEO-M8"
