File: Cowbell_no_gps.sch (KiCad schematic (older format))
At the start: 24 parts, among them J1 Conn_Coaxial, J102 Conn_01x02_Male, J104 Conn_01x02_Male, J105 Conn_01x02_Male, J401 Conn_Coaxial, Q102 DMG6601LVT, U101 SIM28ML, U102 LSM303C, U103 ESP32-WROOM-32, U104 RN2483A-I

Commit message: Updated to newest version
Parts:
- removed J1: Conn_Coaxial, Emborg:u.fl, symbol Connector:Conn_Coaxial
- removed J102: Conn_01x02_Male, Pin_Headers:Pin_Header_Straight_1x02_Pitch2.54mm, symbol Connector:Conn_01x02_Male
- removed L101: >27nH, Inductor_SMD:L_0402_1005Metric, symbol Device:L
- removed Q102: DMG6601LVT, Emborg:DMG6601LVT, symbol Emborg:DMG6601LVT
- removed R101: 10k, Resistor_SMD:R_0603_1608Metric_Pad1.05x0.95mm_HandSolder, symbol Device:R
- removed R102: 10ohm, Resistor_SMD:R_0603_1608Metric_Pad1.05x0.95mm_HandSolder, symbol Device:R
- removed U101: SIM28ML, Emborg:SIM28ML, symbol Emborg:SIM28ML
- added R104, R105, R106: shunt, Resistors_SMD:R_0603, symbol Device:R
- J101: renamed from J401; footprint Emborg:SMA_EdgeMount -> Connectors_Molex:Molex_SMA_Jack_Edge_Mount
- R101: renamed from R401; footprint Resistor_SMD:R_0603_1608Metric -> Resistors_SMD:R_0603_HandSoldering
- R102: renamed from R302; footprint Resistor_SMD:R_0603_1608Metric -> Resistors_SMD:R_0603
- R107: renamed from R307; footprint Resistor_SMD:R_0603_1608Metric -> Resistors_SMD:R_0603
- R201, R202: footprint Resistor_SMD:R_0603_1608Metric -> Resistors_SMD:R_0603
Connections:
- net labels removed: VCC101, VccGPS_backup
- wire segments 122 -> 114
- no-connect marks 5 -> 0
Other:
- note removed: "GPS"
