File: noname1.1.kicad_pcb (KiCad board)
At the start: 2 copper layers, 23.7 x 53.5 mm, 25 parts, among them J1 Conn_Coaxial, J101 Conn_Coaxial, J102 Conn_01x02_Male, J104 Conn_01x02_Male, J105 Conn_01x02_Male, U101 NEO-M8, U102 LSM303C, U103 ESP32-WROOM-32, U104 RN2483A-I

Commit message: Updated to newest version
Routing:
- net SCL: track 46.6 -> 43.4 mm
- net Tx0: track 17.9 -> 20.3 mm
- net /VccGPS_backup: track 18.7 -> 21.0 mm
- net Net-(J105-Pad1): track 28.5 -> 30.7 mm
- net SDA: track 47.4 -> 45.8 mm
- net Rx0: track 14.0 -> 15.6 mm
- net Tx1: track 9.92 -> 8.39 mm
- net Rx1: track 8.66 -> 7.74 mm
- net Net-(C202-Pad1): track 25.2 -> 24.4 mm
- net /VCC103: track 40.0 -> 39.3 mm
- net Timepulse: track 29.1 -> 28.4 mm
- net GND: vias 80 -> 82
Other:
- rule via_min_drill: 0.254 -> 0.305
- board text added: "+ Batt -"
- board text added: "BackUp Batt"
- board text removed: "18650?"
