File: Cowbell_mini.kicad_pcb (KiCad board)
At the start: 2 copper layers, 24.2 x 36.2 mm, 29 parts, among them J101 Conn_Coaxial, J102 Conn_01x02_Male, J104 Conn_01x02_Male, J105 Conn_01x02_Male, J401 Conn_Coaxial, Q102 SOT-23-6, U101 SIM28ML, U102 LSM303C, U103 ESP32-WROOM-32, U105 RFM9x, U5 TPS63001

Commit message: finished design
Parts:
- moved L101 0.33 mm to (122.6, 60.2)
Routing:
- net GND: track 115.2 -> 118.5 mm, vias 120 -> 132
- net +3V3: track 87.2 -> 85.6 mm, vias 9 -> 11
Other:
- board text added: "GND"
- board text added: "VCCGPS_Backup"

Commit message: Final version
Routing:
- net GND: vias 132 -> 131
Changed lines of the file:
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@@
     (thickness 1.6)
     (drawings 23)
-    (tracks 662)
+    (tracks 661)
     (zones 0)
     (modules 29)
@@
       (drillshape 0)
       (scaleselection 1)
-      (outputdirectory ""))
+      (outputdirectory "Gerberfiles_Cow_mini/"))
   )
   (net 0 "")
@@
   (via (at 137.39198 61.82594) (size 0.6858) (drill 0.3302) (layers F.Cu B.Cu) (net 1))
   (via (at 137.13544 55.70454) (size 0.6858) (drill 0.3302) (layers F.Cu B.Cu) (net 1))
-  (via (at 134.26524 31.23672) (size 0.6858) (drill 0.3302) (layers F.Cu B.Cu) (net 1))
   (via (at 128.21496 35.65378) (size 0.6858) (drill 0.3302) (layers F.Cu B.Cu) (net 1))
   (via (at 132.0656 39.2174) (size 0.6858) (drill 0.3302) (layers F.Cu B.Cu) (net 1))
@@
   (segment (start 116.586 35.9664) (end 117.74 34.8124) (width 0.254) (layer B.Cu) (net 33))
   (segment (start 117.74 34.62) (end 117.74 33.8325) (width 0.254) (layer B.Cu) (net 33))
-  (segment (start 134.25 35.89) (end 134.25 32.334) (width 1.25) (layer B.Cu) (net 34))
+  (segment (start 134.25 35.89) (end 134.25 32.334) (width 1.2) (layer B.Cu) (net 34))
   (segment (start 134.13 36.002) (end 133.996 36.144) (width 0.75) (layer B.Cu) (net 34))
   (segment (start 133.996 36.144) (end 134.25 35.89) (width 0.75) (layer B.Cu) (net 34))
@@
   (segment (start 128.377101 56.093101) (end 128.377101 54.909101) (width 0.254) (layer F.Cu) (net 55))
   (segment (start 120.131 61.077) (end 120.073 61.135) (width 0.508) (layer B.Cu) (net 56) (status 30))
-  (segment (start 125.844 61.034) (end 120.002 61.034) (width 1.25) (layer B.Cu) (net 56))
+  (segment (start 125.844 61.034) (end 120.002 61.034) (width 1.2) (layer B.Cu) (net 56))
   (segment (start 118.5 46.16) (end 119.182922 46.16) (width 0.254) (layer F.Cu) (net 57))
   (via (at 122.05801 42.24) (size 0.6858) (drill 0.3302) (layers F.Cu B.Cu) (net 57))
